File: board/mnhttn.kicad_pcb (KiCad board)
At the start: 2 copper layers, 257.8 x 89.2 mm, 82 parts, among them SW1 SW_Push, SW2 SW_SPDT, SW3 SW_Push, SW4 SW_SPDT, U1 xiao-ble, U2 xiao-ble

Commit message: Add battery connector
Parts:
- removed BAT+1, BAT+2: +, mnhttn:BatteryPad
- removed BAT-1, BAT-2: -, mnhttn:BatteryPad
- added BT1: Battery_Cell, mnhttn:WAGO_2060-452_998-404, F.Cu at (81.3, 105.4)
- added BT2: Battery_Cell, mnhttn:WAGO_2060-452_998-404, F.Cu at (217.2, 105.4)
- moved SW_R_0_3 1.27 mm to (162.6, 110.4)
- moved SW_R_1_3 1.12 mm to (182.2, 104.7)
- moved SW_R_2_3 1.12 mm to (202.6, 104.7)
Connections:
- D_L_0_0 pad 1: /ROW_0_L -> /Switch4/ROW
- D_L_0_1 pad 1: /ROW_1_L -> /Switch5/ROW
- D_L_0_2 pad 1: /ROW_2_L -> /Switch13/ROW
- D_L_0_3 pad 1: /ROW_3_L -> /Switch17/ROW
- D_L_1_0 pad 1: /ROW_0_L -> /Switch3/ROW
- D_L_1_1 pad 1: /ROW_1_L -> /Switch7/ROW
- D_L_1_2 pad 1: /ROW_2_L -> /Switch11/ROW
- D_L_1_3 pad 1: /ROW_3_L -> /Switch16/ROW
- D_L_2_0 pad 1: /ROW_0_L -> /Switch2/ROW
- D_L_2_1 pad 1: /ROW_1_L -> /Switch9/ROW
- D_L_2_2 pad 1: /ROW_2_L -> /Switch12/ROW
- D_L_3_0 pad 1: /ROW_0_L -> /Switch1/ROW
- D_L_3_1 pad 1: /ROW_1_L -> /Switch8/ROW
- D_L_3_2 pad 1: /ROW_2_L -> /Switch10/ROW
- D_R_0_0 pad 1: /ROW_0_R -> /Switch20/ROW
- D_R_0_1 pad 1: /ROW_1_R -> /Switch23/ROW
- D_R_0_2 pad 1: /ROW_2_R -> /Switch22/ROW
- D_R_0_3 pad 1: /ROW_3_R -> /Switch29/ROW
- D_R_1_0 pad 1: /ROW_0_R -> /Switch19/ROW
- D_R_1_1 pad 1: /ROW_1_R -> /Switch18/ROW
- D_R_1_2 pad 1: /ROW_2_R -> /Switch21/ROW
- D_R_1_3 pad 1: /ROW_3_R -> /Switch31/ROW
- D_R_2_0 pad 1: /ROW_0_R -> /Switch24/ROW
- D_R_2_1 pad 1: /ROW_1_R -> /Switch26/ROW
- D_R_2_2 pad 1: /ROW_2_R -> /Switch25/ROW
- D_R_3_0 pad 1: /ROW_0_R -> /Switch27/ROW
- D_R_3_1 pad 1: /ROW_1_R -> /Switch32/ROW
- D_R_3_2 pad 1: /ROW_2_R -> /Switch35/ROW
- SW_L_0_0 pad 2: /COL_0_L -> /Switch4/COL
- SW_L_0_1 pad 2: /COL_0_L -> /Switch5/COL
- SW_L_0_2 pad 2: /COL_0_L -> /Switch13/COL
- SW_L_1_0 pad 2: /COL_1_L -> /Switch3/COL
- SW_L_1_1 pad 2: /COL_1_L -> /Switch7/COL
- SW_L_1_2 pad 2: /COL_1_L -> /Switch11/COL
- SW_L_2_0 pad 2: /COL_2_L -> /Switch2/COL
- SW_L_2_1 pad 2: /COL_2_L -> /Switch9/COL
- SW_L_2_2 pad 2: /COL_2_L -> /Switch12/COL
- SW_L_3_0 pad 2: /COL_3_L -> /Switch1/COL
- SW_L_3_1 pad 2: /COL_3_L -> /Switch8/COL
- SW_L_4_0 pad 2: /COL_4_L -> /Switch/COL
- SW_L_4_1 pad 2: /COL_4_L -> /Switch6/COL
- SW_R_0_0 pad 2: /COL_0_R -> /Switch20/COL
- SW_R_0_1 pad 2: /COL_0_R -> /Switch23/COL
- SW_R_0_2 pad 2: /COL_0_R -> /Switch22/COL
- SW_R_1_0 pad 2: /COL_1_R -> /Switch19/COL
- SW_R_1_1 pad 2: /COL_1_R -> /Switch18/COL
- SW_R_1_2 pad 2: /COL_1_R -> /Switch21/COL
- SW_R_2_0 pad 2: /COL_2_R -> /Switch24/COL
- SW_R_2_1 pad 2: /COL_2_R -> /Switch26/COL
- SW_R_2_2 pad 2: /COL_2_R -> /Switch25/COL
- SW_R_3_0 pad 2: /COL_3_R -> /Switch27/COL
- SW_R_3_1 pad 2: /COL_3_R -> /Switch32/COL
- SW_R_4_0 pad 2: /COL_4_R -> /Switch28/COL
- SW_R_4_1 pad 2: /COL_4_R -> /Switch34/COL
Routing:
- net -BATT: track 193.0 -> 222.4 mm
- net Net-(BT2-+): track 99.2 -> 116.7 mm, vias 2 -> 4
- net Net-(BT1-+): track 96.5 -> 113.3 mm
- net Net-(D_R_0_3-A): track 25.6 -> 27.2 mm
- net /COL_0_R: track 164.0 -> 165.3 mm
- net /COL_1_R: track 147.8 -> 149.0 mm
- net Net-(D_R_2_3-A): track 30.2 -> 29.1 mm
- net Net-(D_R_1_3-A): track 15.1 -> 14.0 mm
- net /COL_2_R: track 119.6 -> 120.2 mm
Other:
- outline, holes or cut-outs redrawn

Commit message: SMD only, On/Off symbole, Cleanup
Parts:
- U1, U2: footprint mnhttn:xiao-ble-smd-cutout -> mnhttn:xiao-ble-smd
Connections:
- D_L_0_0 pad 1: /Switch4/ROW -> /ROW_0_L
- D_L_0_1 pad 1: /Switch5/ROW -> /ROW_1_L
- D_L_0_2 pad 1: /Switch13/ROW -> /ROW_2_L
- D_L_0_3 pad 1: /Switch17/ROW -> /ROW_3_L
- D_L_1_0 pad 1: /Switch3/ROW -> /ROW_0_L
- D_L_1_1 pad 1: /Switch7/ROW -> /ROW_1_L
- D_L_1_2 pad 1: /Switch11/ROW -> /ROW_2_L
- D_L_1_3 pad 1: /Switch16/ROW -> /ROW_3_L
- D_L_2_0 pad 1: /Switch2/ROW -> /ROW_0_L
- D_L_2_1 pad 1: /Switch9/ROW -> /ROW_1_L
- D_L_2_2 pad 1: /Switch12/ROW -> /ROW_2_L
- D_L_3_0 pad 1: /Switch1/ROW -> /ROW_0_L
- D_L_3_1 pad 1: /Switch8/ROW -> /ROW_1_L
- D_L_3_2 pad 1: /Switch10/ROW -> /ROW_2_L
- D_R_0_0 pad 1: /Switch20/ROW -> /ROW_0_R
- D_R_0_1 pad 1: /Switch23/ROW -> /ROW_1_R
- D_R_0_2 pad 1: /Switch22/ROW -> /ROW_2_R
- D_R_0_3 pad 1: /Switch29/ROW -> /ROW_3_R
- D_R_1_0 pad 1: /Switch19/ROW -> /ROW_0_R
- D_R_1_1 pad 1: /Switch18/ROW -> /ROW_1_R
- D_R_1_2 pad 1: /Switch21/ROW -> /ROW_2_R
- D_R_1_3 pad 1: /Switch31/ROW -> /ROW_3_R
- D_R_2_0 pad 1: /Switch24/ROW -> /ROW_0_R
- D_R_2_1 pad 1: /Switch26/ROW -> /ROW_1_R
- D_R_2_2 pad 1: /Switch25/ROW -> /ROW_2_R
- D_R_3_0 pad 1: /Switch27/ROW -> /ROW_0_R
- D_R_3_1 pad 1: /Switch32/ROW -> /ROW_1_R
- D_R_3_2 pad 1: /Switch35/ROW -> /ROW_2_R
- SW_L_0_0 pad 2: /Switch4/COL -> /COL_0_L
- SW_L_0_1 pad 2: /Switch5/COL -> /COL_0_L
- SW_L_0_2 pad 2: /Switch13/COL -> /COL_0_L
- SW_L_1_0 pad 2: /Switch3/COL -> /COL_1_L
- SW_L_1_1 pad 2: /Switch7/COL -> /COL_1_L
- SW_L_1_2 pad 2: /Switch11/COL -> /COL_1_L
- SW_L_2_0 pad 2: /Switch2/COL -> /COL_2_L
- SW_L_2_1 pad 2: /Switch9/COL -> /COL_2_L
- SW_L_2_2 pad 2: /Switch12/COL -> /COL_2_L
- SW_L_3_0 pad 2: /Switch1/COL -> /COL_3_L
- SW_L_3_1 pad 2: /Switch8/COL -> /COL_3_L
- SW_L_4_0 pad 2: /Switch/COL -> /COL_4_L
- SW_L_4_1 pad 2: /Switch6/COL -> /COL_4_L
- SW_R_0_0 pad 2: /Switch20/COL -> /COL_0_R
- SW_R_0_1 pad 2: /Switch23/COL -> /COL_0_R
- SW_R_0_2 pad 2: /Switch22/COL -> /COL_0_R
- SW_R_1_0 pad 2: /Switch19/COL -> /COL_1_R
- SW_R_1_1 pad 2: /Switch18/COL -> /COL_1_R
- SW_R_1_2 pad 2: /Switch21/COL -> /COL_1_R
- SW_R_2_0 pad 2: /Switch24/COL -> /COL_2_R
- SW_R_2_1 pad 2: /Switch26/COL -> /COL_2_R
- SW_R_2_2 pad 2: /Switch25/COL -> /COL_2_R
- SW_R_3_0 pad 2: /Switch27/COL -> /COL_3_R
- SW_R_3_1 pad 2: /Switch32/COL -> /COL_3_R
- SW_R_4_0 pad 2: /Switch28/COL -> /COL_4_R
- SW_R_4_1 pad 2: /Switch34/COL -> /COL_4_R
Routing:
- net /ROW_3_R: track 146.6 -> 145.3 mm, vias 1 -> 2
- net Net-(BT2-+): track 116.7 -> 117.9 mm
- net /ROW_3_L: vias 1 -> 2
- net /ROW_1_R: vias 1 -> 2
- net /RST_L: vias 1 -> 2
- net /ROW_0_L: vias 1 -> 2
- net /ROW_0_R: vias 1 -> 2
- net GND: vias 9 -> 16
- net /RST_R: vias 1 -> 2
- net /ROW_2_R: vias 1 -> 2
- net /ROW_2_L: vias 1 -> 2
- net /ROW_1_L: vias 1 -> 2
Other:
- outline, holes or cut-outs redrawn
- board text added: "rev. 0003 by fooker"
- board text removed: "rev. 0002 by fooker"
